Commit message: fiexed launch files

File: bot_with_camera/urdf/cam.urdf.xacro (robot description, xacro)
@@ -34,5 +34,5 @@
 </link>
 <joint name="joint_name" type="fixed">
-    <parent link="base_link"/>
+    <parent link="base_footprint"/>
     <child link="camera_link"/>
     <origin xyz="0.03 0.0 ${bot_height}" rpy="0.0 0.0 0.0"/>

Commit message: changed some parameters,still camera plugin not visible in gazebo GUI

File: bot_with_camera/urdf/cam.urdf.xacro (robot description, xacro)
@@ -2,5 +2,5 @@
 <robot xmlns:xacro="http://www.ros.org/wiki/xacro" name="turtlebot">
 <xacro:include filename="$(find bot_with_camera)/urdf/cam.gazebo"/>
-<xacro:property name="bot_height" value="0.15"/>
+<xacro:property name="bot_height" value="0.14"/>
 <xacro:property name="cam_length" value="0.005"/>
 <xacro:property name="cam_width" value="0.01"/>
@@ -34,7 +34,8 @@
 </link>
 <joint name="joint_name" type="fixed">
-    <parent link="base_footprint"/>
+    <axis xyz="0 1 0"/>
+    <parent link="base_link"/>
     <child link="camera_link"/>
-    <origin xyz="0.03 0.0 ${bot_height}" rpy="0.0 0.0 0.0"/>
+    <origin xyz="0.032 0.0 ${bot_height}" rpy="0.0 0.0 0.0"/>
 </joint>
 </robot>
